File: KiCad/HagiwoEurorackMixer_PCBOnly.kicad_pcb (KiCad board)
At the start: 2 copper layers, 66 x 128.5 mm, 34 parts, among them J1 IN 1, J2 IN 2, J3 IN 3, J4 IN 4, J5 OUT, J6 EURO_PWR_2x5, U2 TL072

Commit message: Produced separate front panel and PCB gerber files for manufacture
Parts:
- removed REF** (x10): MountingHole_6mm, Library:MountingHole_6mm
- removed REF** (x2): Eurorack_Panel_ScrewHole_Oval, Library:Eurorack_Panel_ScrewHole_Oval
Other:
- board size 66 x 128.5 mm -> 29 x 106 mm
- board text added: "V1.0: PCB + PANEL BY 42 BERLIN SYNTHLAB https://workish.berlin/fablab"
- board text removed: "1"
- board text removed: "2"
- board text removed: "3"
- board text removed: "4"
- board text removed: "CONCRETE MIXER"
- board text removed: "IN"
- board text removed: "LEVEL"
- board text removed: "OUT"
- board text removed: "SynthLab"

Commit message: Produced files for uploading to jlcpcb - first attempt
Other:
- board text added: "JLCJLCJLCJLC"
- board text removed: "PCB + PANEL BY 42 BERLIN SYNTHLAB https://workish.berlin/fablab"
