File: KiCad/HagiwoEurorackMixer_PanelOnly.kicad_pcb (KiCad board)
At the start: 2 copper layers, 30 x 128.5 mm, 12 parts

Commit message: Produced files for uploading to jlcpcb - first attempt
Other:
- board text added: "JLCJLCJLCJLC"
- board text removed: "ORIGINAL DESIGN BY HAGIWO / DOEPFER"
- board text removed: "PCB + PANEL BY 42 BERLIN SYNTHLAB https://workish.berlin/fablab"
