File: HagiwoEurorackMixer.kicad_pcb (KiCad board)
At the start: 2 copper layers, 29 x 106 mm, 22 parts, among them J1 IN1, J2 IN2, J3 IN3, J4 IN4, J5 OUT, J7 Eurorack_Power_10pin_Unshroud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, U2 TL072

Commit message: v1.2 ready for production - slightly unsure if volume pot left/right side wiring is correct
Parts:
- added D1: 1N5817, Diode_THT:D_DO-41_SOD81_P10.16mm_Horizontal, B.Cu at (79.0, 130.0)
- added D2: 1N5817, Diode_THT:D_DO-41_SOD81_P10.16mm_Horizontal, B.Cu at (79.0, 133.3)
- moved R8 17.0 mm to (90.1, 147.4), turned to 0 degrees
- moved R7 10.4 mm to (87.6, 126.8), turned to 180 degrees
- moved C1 1.35 mm to (103.1, 148.9)
- moved C2 0.61 mm to (103.1, 156.2)
Connections:
- C1 pad 1: Net-(U2C-V+) -> Net-(D1-K)
- C2 pad 2: Net-(U2C-V-) -> Net-(D2-A)
- J7 pad 1: Net-(U2C-V+) -> Net-(D1-A)
- J7 pad 10: Net-(U2C-V-) -> Net-(D2-K)
- J7 pad 2: Net-(U2C-V+) -> Net-(D1-A)
- J7 pad 9: Net-(U2C-V-) -> Net-(D2-K)
- RV1 pad 1: Net-(J1-PadT) -> GND
- RV1 pad 3: GND -> Net-(J1-PadT)
- RV2 pad 1: Net-(J2-PadT) -> GND
- RV2 pad 3: GND -> Net-(J2-PadT)
- RV3 pad 1: Net-(J3-PadT) -> GND
- RV3 pad 3: GND -> Net-(J3-PadT)
- RV4 pad 1: Net-(J4-PadT) -> GND
- RV4 pad 3: GND -> Net-(J4-PadT)
- RV5 pad 1: Net-(U2B--) -> Net-(R7-Pad1)
- RV5 pad 3: Net-(R7-Pad1) -> Net-(U2B--)
- U2 pad 4: Net-(U2C-V-) -> Net-(D2-A)
- U2 pad 8: Net-(U2C-V+) -> Net-(D1-K)
Routing:
- net Net-(U2C-V-): track 75.8 -> 0.00 mm
- net Net-(D2-A): track 0.00 -> 68.5 mm, vias 0 -> 7
- net Net-(U2C-V+): track 57.9 -> 0.00 mm
- net Net-(D1-K): track 0.00 -> 51.6 mm, vias 0 -> 4
- net Net-(D1-A): track 0.00 -> 28.0 mm
- net Net-(D2-K): track 0.00 -> 25.9 mm
- net Net-(J5-PadT): track 29.5 -> 9.19 mm, vias 3 -> 0
- net Net-(R7-Pad2): track 22.5 -> 39.9 mm, vias 1 -> 2
- net Net-(U2B--): track 58.4 -> 48.2 mm
- net Net-(J3-PadT): track 20.8 -> 25.9 mm
- net Net-(J2-PadT): track 20.8 -> 25.9 mm
- net Net-(J1-PadT): track 20.8 -> 25.9 mm
- net Net-(J4-PadT): track 21.1 -> 25.9 mm
- net Net-(U2A--): track 98.6 -> 99.4 mm, vias 1 -> 2
- net Net-(R7-Pad1): track 24.7 -> 25.5 mm, vias 0 -> 1
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Other:
- board text added: "V1.2"
- board text added: "https://www.github.com/fablabnk/ SynthLabProjects"
- board text removed: "V1.1"
- board text removed: "github.com/fablabnk/SynthLabProjects"
